File: floppy-drives/direct-drive/direct-drive.kicad_pcb (KiCad board)
At the start: 2 copper layers, 27.7 x 51.1 mm, 18 parts, among them J1 Floppy Drive, J2 Control, SW1 Reset, SW2 User, U1 ATtiny24A-P, U2 TXU0304PWR, Y1 ASEM1-8.000MHZ

Commit message: direct-drive: Move oscillator a little closer to the chip
Parts:
- moved Y1 1.08 mm to (132.2, 64.5)
- moved C2 0.38 mm to (132.5, 67.6)
Routing:
- net +3V3: track 77.5 -> 80.1 mm
Changed lines of the file:
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@@
   (net 36 "DRVS-L")
   (footprint "Capacitor_SMD:C_0603_1608Metric" (layer "F.Cu")
-    (at 132.842 67.564)
+    (at 132.461 67.564)
     (descr "Capacitor SMD 0603 (1608 Metric), square (rectangular) end terminal, IPC_7351 nominal, (Body size source: IPC-SM-782 page 76, https://www.pcb-3d.com/wordpress/wp-content/uploads/ipc-sm-782a_amendment_1_and_2.pdf), generated with kicad-footprint-generator")
     (tags "capacitor")
@@
     (property "Sheetname" "")
     (attr smd)
-    (fp_text reference "C2" (at 0 1.778 90) (layer "F.SilkS")
+    (fp_text reference "C2" (at 0.635 2.159 90) (layer "F.SilkS")
       (effects (font (size 1 1) (thickness 0.15)))
     )
@@
     (property "Sheetname" "")
     (attr smd)
-    (fp_text reference "C1" (at 0 -1.43 90) (layer "F.SilkS")
+    (fp_text reference "C1" (at 0.381 -1.43 90) (layer "F.SilkS")
       (effects (font (size 1 1) (thickness 0.15)))
     )
@@
   )
   (footprint "agausmann:ASEM-4Pin-3.2x2.5mm" (layer "F.Cu")
-    (at 133.284 64.55 90)
+    (at 132.207 64.55 90)
     (property "Digikey" "535-9754-1-ND")
     (property "Sheetfile" "direct-drive.kicad_sch")
     (property "Sheetname" "")
     (attr smd)
-    (fp_text reference "Y1" (at -0.982 2.606 90 unlocked) (layer "F.SilkS")
+    (fp_text reference "Y1" (at 1.177 2.667 90 unlocked) (layer "F.SilkS")
       (effects (font (size 1 1) (thickness 0.15)))
     )
@@
   (segment (start 133.35 49.096) (end 133.058 48.804) (width 0.4) (layer "F.Cu") (net 1))
   (segment (start 129.54 66.04) (end 129.54 68.059) (width 0.4) (layer "F.Cu") (net 1))
-  (segment (start 132.067 67.564) (end 132.067 65.867) (width 0.4) (layer "F.Cu") (net 1))
+  (segment (start 133.157 65.6) (end 133.157 66.093) (width 0.4) (layer "F.Cu") (net 1))
   (segment (start 122.391427 68.662) (end 121.5975 68.662) (width 0.4) (layer "F.Cu") (net 1))
-  (segment (start 132.067 67.831) (end 131.318 68.58) (width 0.4) (layer "F.Cu") (net 1))
-  (segment (start 130.048 68.567) (end 131.305 68.567) (width 0.4) (layer "F.Cu") (net 1))
+  (segment (start 131.257 67.135) (end 131.686 67.564) (width 0.4) (layer "F.Cu") (net 1))
+  (segment (start 131.257 65.6) (end 131.257 67.135) (width 0.4) (layer "F.Cu") (net 1))
+  (segment (start 131.686 67.564) (end 131.686 68.212) (width 0.4) (layer "F.Cu") (net 1))
   (segment (start 127.521 74.422) (end 127.521 72.7605) (width 0.4) (layer "F.Cu") (net 1))
-  (segment (start 132.067 67.564) (end 132.067 67.831) (width 0.4) (layer "F.Cu") (net 1))
+  (segment (start 131.686 68.212) (end 131.191 68.707) (width 0.4) (layer "F.Cu") (net 1))
+  (segment (start 130.188 68.707) (end 130.048 68.567) (width 0.4) (layer "F.Cu") (net 1))
   (segment (start 126.291427 72.562) (end 122.391427 68.662) (width 0.4) (layer "F.Cu") (net 1))
   (segment (start 141.008 48.804) (end 133.058 48.804) (width 0.4) (layer "F.Cu") (net 1))
-  (segment (start 134.234 65.6) (end 134.615 65.6) (width 0.4) (layer "F.Cu") (net 1))
   (segment (start 129.54 68.059) (end 130.048 68.567) (width 0.4) (layer "F.Cu") (net 1))
-  (segment (start 134.234 65.6) (end 134.234 65.603596) (width 0.4) (layer "F.Cu") (net 1))
-  (segment (start 131.305 68.567) (end 131.318 68.58) (width 0.4) (layer "F.Cu") (net 1))
-  (segment (start 132.067 65.867) (end 132.334 65.6) (width 0.4) (layer "F.Cu") (net 1))
+  (segment (start 136.398 63.817) (end 136.081 63.817) (width 0.4) (layer "F.Cu") (net 1))
+  (segment (start 131.191 68.707) (end 130.188 68.707) (width 0.4) (layer "F.Cu") (net 1))
+  (segment (start 136.081 63.817) (end 134.62 65.278) (width 0.4) (layer "F.Cu") (net 1))
   (segment (start 136.906 75.8365) (end 131.4625 81.28) (width 0.4) (layer "F.Cu") (net 1))
-  (segment (start 134.234 65.603596) (end 133.34686 66.490736) (width 0.4) (layer "F.Cu") (net 1))
+  (segment (start 133.157 66.093) (end 131.686 67.564) (width 0.4) (layer "F.Cu") (net 1))
   (segment (start 136.906 72.707) (end 136.906 75.8365) (width 0.4) (layer "F.Cu") (net 1))
   (segment (start 127.3225 72.562) (end 126.291427 72.562) (width 0.4) (layer "F.Cu") (net 1))
   (segment (start 133.35 50.292) (end 133.35 49.096) (width 0.4) (layer "F.Cu") (net 1))
-  (segment (start 134.615 65.6) (end 136.398 63.817) (width 0.4) (layer "F.Cu") (net 1))
   (segment (start 127.521 72.7605) (end 127.3225 72.562) (width 0.4) (layer "F.Cu") (net 1))
-  (via (at 133.34686 66.490736) (size 0.8) (drill 0.4) (layers "F.Cu" "B.Cu") (net 1))
+  (via (at 134.62 65.278) (size 0.8) (drill 0.4) (layers "F.Cu" "B.Cu") (net 1))
   (via (at 127.762 75.692) (size 0.8) (drill 0.4) (layers "F.Cu" "B.Cu") (net 1))
+  (via (at 131.191 68.707) (size 0.8) (drill 0.4) (layers "F.Cu" "B.Cu") (net 1))
   (via (at 133.35 50.292) (size 0.8) (drill 0.4) (layers "F.Cu" "B.Cu") (net 1))
-  (via (at 131.318 68.58) (size 0.8) (drill 0.4) (layers "F.Cu" "B.Cu") (net 1))
+  (segment (start 133.35 50.292) (end 133.312489 50.329511) (width 0.4) (layer "B.Cu") (net 1))
   (segment (start 131.4625 81.28) (end 131.4625 79.3925) (width 0.4) (layer "B.Cu") (net 1))
   (segment (start 131.4625 79.3925) (end 127.762 75.692) (width 0.4) (layer "B.Cu") (net 1))
-  (segment (start 133.34686 66.490736) (end 133.34686 66.55114) (width 0.4) (layer "B.Cu") (net 1))
-  (segment (start 133.312489 66.456365) (end 133.312489 50.329511) (width 0.4) (layer "B.Cu") (net 1))
-  (segment (start 133.34686 66.490736) (end 133.312489 66.456365) (width 0.4) (layer "B.Cu") (net 1))
-  (segment (start 133.312489 50.329511) (end 133.35 50.292) (width 0.4) (layer "B.Cu") (net 1))
-  (segment (start 127.762 75.692) (end 127.762 72.136) (width 0.4) (layer "B.Cu") (net 1))
-  (segment (start 127.762 72.136) (end 131.318 68.58) (width 0.4) (layer "B.Cu") (net 1))
-  (segment (start 133.34686 66.55114) (end 131.318 68.58) (width 0.4) (layer "B.Cu") (net 1))
+  (segment (start 133.312489 66.585511) (end 134.62 65.278) (width 0.4) (layer "B.Cu") (net 1))
+  (segment (start 133.312489 66.585511) (end 127.762 72.136) (width 0.4) (layer "B.Cu") (net 1))
+  (segment (start 127.762 72.136) (end 127.762 75.692) (width 0.4) (layer "B.Cu") (net 1))
+  (segment (start 133.312489 50.329511) (end 133.312489 66.585511) (width 0.4) (layer "B.Cu") (net 1))
   (segment (start 127.3225 68.3945) (end 126.746 67.818) (width 0.4) (layer "F.Cu") (net 2))
   (segment (start 138.9635 72.6695) (end 139.446 73.152) (width 0.4) (layer "F.Cu") (net 2))
   (segment (start 133.058 55.662) (end 134.529 55.662) (width 0.4) (layer "F.Cu") (net 2))
   (segment (start 130.048 70.117) (end 130.048 71.247) (width 0.4) (layer "F.Cu") (net 2))
-  (segment (start 133.617 67.564) (end 133.617 68.821) (width 0.4) (layer "F.Cu") (net 2))
   (segment (start 122.695 74.422) (end 122.695 73.346237) (width 0.4) (layer "F.Cu") (net 2))
   (segment (start 125.971 73.927) (end 126.492 73.406) (width 0.4) (layer "F.Cu") (net 2))
   (segment (start 130.048 71.247) (end 130.302 71.501) (width 0.4) (layer "F.Cu") (net 2))
-  (segment (start 134.234 63.5) (end 134.234 62.616) (width 0.4) (layer "F.Cu") (net 2))
+  (segment (start 133.096 63.5) (end 132.08 62.484) (width 0.4) (layer "F.Cu") (net 2))
+  (segment (start 133.236 67.564) (end 133.236 68.694) (width 0.4) (layer "F.Cu") (net 2))
+  (segment (start 133.236 68.694) (end 133.223 68.707) (width 0.4) (layer "F.Cu") (net 2))
   (segment (start 122.695 73.346237) (end 122.616983 73.26822) (width 0.4) (layer "F.Cu") (net 2))
   (segment (start 138.9635 68.0465) (end 139.446 67.564) (width 0.4) (layer "F.Cu") (net 2))
   (segment (start 138.43 68.0465) (end 138.9635 68.0465) (width 0.4) (layer "F.Cu") (net 2))
-  (segment (start 134.234 62.616) (end 134.62 62.23) (width 0.4) (layer "F.Cu") (net 2))
   (segment (start 127.3225 68.662) (end 127.3225 68.3945) (width 0.4) (layer "F.Cu") (net 2))
   (segment (start 138.43 72.6695) (end 138.9635 72.6695) (width 0.4) (layer "F.Cu") (net 2))
   (segment (start 141.008 55.662) (end 134.529 55.662) (width 0.4) (layer "F.Cu") (net 2))
   (segment (start 137.922 63.817) (end 137.922 64.008) (width 0.4) (layer "F.Cu") (net 2))
-  (segment (start 133.617 68.821) (end 133.604 68.834) (width 0.4) (layer "F.Cu") (net 2))
   (segment (start 125.971 74.422) (end 125.971 73.927) (width 0.4) (layer "F.Cu") (net 2))
   (segment (start 137.922 64.008) (end 137.16 64.77) (width 0.4) (layer "F.Cu") (net 2))
+  (segment (start 133.157 63.5) (end 133.096 63.5) (width 0.4) (layer "F.Cu") (net 2))
   (via (at 134.529 55.662) (size 0.8) (drill 0.4) (layers "F.Cu" "B.Cu") (net 2))
-  (via (at 133.604 68.834) (size 0.8) (drill 0.4) (layers "F.Cu" "B.Cu") (net 2))
+  (via (at 133.223 68.707) (size 0.8) (drill 0.4) (layers "F.Cu" "B.Cu") (net 2))
   (via (at 137.16 64.77) (size 0.8) (drill 0.4) (layers "F.Cu" "B.Cu") (net 2))
-  (via (at 134.62 62.23) (size 0.8) (drill 0.4) (layers "F.Cu" "B.Cu") (net 2))
   (via (at 126.746 67.818) (size 0.8) (drill 0.4) (layers "F.Cu" "B.Cu") (net 2))
   (via (at 130.302 71.501) (size 0.8) (drill 0.4) (layers "F.Cu" "B.Cu") (net 2))
@@
   (via (at 122.616983 73.26822) (size 0.8) (drill 0.4) (layers "F.Cu" "B.Cu") (net 2))
   (via (at 126.492 73.406) (size 0.8) (drill 0.4) (layers "F.Cu" "B.Cu") (net 2))
+  (via (at 132.08 62.484) (size 0.8) (drill 0.4) (layers "F.Cu" "B.Cu") (net 2))
   (segment (start 128.9225 83.82) (end 130.1925 85.09) (width 0.4) (layer "B.Cu") (net 2))
   (segment (start 130.1925 85.09) (end 132.588 85.09) (width 0.4) (layer "B.Cu") (net 2))
@@
   (via (at 136.652 60.96) (size 0.8) (drill 0.4) (layers "F.Cu" "B.Cu") (net 29))
   (segment (start 136.652 60.96) (end 135.001 59.309) (width 0.25) (layer "B.Cu") (net 29))
-  (segment (start 132.334 63.5) (end 129.54 63.5) (width 0.25) (layer "F.Cu") (net 30))
+  (segment (start 131.257 63.5) (end 128.905 63.5) (width 0.25) (layer "F.Cu") (net 30))
   (segment (start 126.479154 69.962) (end 123.90356 67.386406) (width 0.25) (layer "F.Cu") (net 33))
   (segment (start 123.90356 67.386406) (end 123.90356 58.49856) (width 0.25) (layer "F.Cu") (net 33))
